File: EggIncubator-Pro-copilot-stabilize-platformio-workflow/hardware/eggincubator-pro.kicad_sch (KiCad schematic)
At the start: 36 parts, among them J10 ESP32 DevKit 5V / VIN input, J11 BTS7960 motor supply input, J2 SHT31 module, I2C 0x44, J3 DS18B20, 1-Wire, J4 4 optocoupled relay-control o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, J5 BTS7960 module / motor (separ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, J6 Door and turner limit switches, J7 5V buzzer module, Q1 low-side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, J8 Expansion: I2C / ADC sensors, J9 12V DC input, Q1 PN2222A, U1 PC817, U2 PC817, U3 PC817, U4 PC817, U5 ESP32 DevKit V1, U9 12V to 5V buck module

Commit message: Correct schematic nets and align wiring guide
Co-authored-by: tomnyle <175001228+tomnyle@users.noreply.github.com>
Connections:
- net 3V3: no longer R1.1
- net ONEWIRE_DQ: no longer R1.2
Changed lines of the file:
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@@
   (label "DEVKIT_5V" (at 324.92 150 180) (fields_autoplaced) (effects (font (size 1.27 1.27)) (justify right bottom)))
   (label "BUZZER_NEG" (at 324.92 152.54 180) (fields_autoplaced) (effects (font (size 1.27 1.27)) (justify right bottom)))
-  (label "3V3" (at 181.19 166 180) (fields_autoplaced) (effects (font (size 1.27 1.27)) (justify right bottom)))
-  (label "ONEWIRE_DQ" (at 188.81 166 0) (fields_autoplaced) (effects (font (size 1.27 1.27)) (justify left bottom)))
+  (label "3V3" (at 185 162.19 180) (fields_autoplaced) (effects (font (size 1.27 1.27)) (justify right bottom)))
+  (label "ONEWIRE_DQ" (at 185 169.81 0) (fields_autoplaced) (effects (font (size 1.27 1.27)) (justify left bottom)))
   (label "3V3" (at 246.19 52.46 180) (fields_autoplaced) (effects (font (size 1.27 1.27)) (justify right bottom)))
   (label "OPTO_HEAT_A" (at 253.81 52.46 0) (fields_autoplaced) (effects (font (size 1.27 1.27)) (justify left bottom)))
